File: FanDC-DC.kicad_sch (KiCad schematic)
At the start: 15 parts, among them IC4 TPS56A37RPAR, J4 Conn_01x02

Commit message: Charging circuit, new block diagram, MCU and display
Parts:
- removed D4: LED, symbol Device:LED
- removed R16: 10k, symbol Device:R
- removed R17: 100k, symbol Device:R
- added D3: LED, symbol lib:LED
- added Q3: 2N7002_SOT-23-3, Hardware Components Footprints:SOT-23-3, symbol lib:2N7002_SOT-23-3
- added R17: R_0R_0402, Hardware Components Footprints:R_0402_1005Metric, symbol lib:R_0R_0402
- added R18, R19: TBD, symbol lib:R_Small
- added R23: 100k, symbol lib:R
- added R24: R_1k_0201, Hardware Components Footprints:R_0201, symbol lib:R_1k_0201
- C10: renamed from C14; symbol Device:C -> lib:C
- C11: renamed from C17; symbol Device:C -> lib:C
- C12: renamed from C15; symbol Device:C -> lib:C
- C13: renamed from C16; symbol Device:C -> lib:C
- C9: renamed from C13; symbol Device:C -> lib:C
- Cboot3: symbol Device:C -> lib:C
- IC3: renamed from IC4; symbol DC-DC converters:TPS56A37RPAR -> lib:TPS56A37RPAR
- J3: renamed from J4; symbol Connector_Generic:Conn_01x02 -> lib:Conn_01x02
- L3: renamed from L4; symbol Device:L -> lib:L
- R20: renamed from R18; symbol Device:R -> lib:R
- R21: renamed from R19; symbol Device:R -> lib:R
- R22: renamed from R20; symbol Device:R -> lib:R
Connections:
- net +16V: now also R18.1, R23.2, R24.2
- net GND: now also Q3.2 (S), R19.2
- net at IC3.1 (EN): now also R17.2, R18.2, R19.1
- net pg_fan: now reaches IC3.4 (PG)
- net pg_fan: now also Q3.1 (G), R23.1
- new net: D3.1 (K), Q3.3 (D)
- new net: D3.2 (A), R24.1
- new net fan_en : R17.1
Other:
- moved on the sheet: C10, C11, C12, C13, C9, Cboot3, IC3, J3, L3, R20, R21, R22

Commit message: Clean up
Other:
- title: (none) -> Robot power supply
Changed lines of the file:
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@@
 	(generator_version "9.0")
 	(paper "A4")
+	(title_block
+		(title "Robot power supply")
+		(date "2026-01-24")
+		(rev "rev 1.0")
+	)
 	(junction
 		(at 248.92 109.22)
