File: GasDC-DC.kicad_sch (KiCad schematic)
At the start: 14 parts, among them IC2 TPS56637RPAR, J1 Conn_01x02

Commit message: Charging circuit, new block diagram, MCU and display
Parts:
- removed R5: 10k, symbol Device:R
- added Q1: 2N7002_SOT-23-3, Hardware Components Footprints:SOT-23-3, symbol lib:2N7002_SOT-23-3
- added R1: R_0R_0402, Hardware Components Footprints:R_0402_1005Metric, symbol lib:R_0R_0402
- added R2, R3: TBD, symbol lib:R_Small
- added R8: R_1k_0201, Hardware Components Footprints:R_0201, symbol lib:R_1k_0201
- C1: renamed from C4; symbol Device:C -> lib:C
- C2: renamed from C5; symbol Device:C -> lib:C
- C3: renamed from C2; symbol Device:C -> lib:C
- C4: renamed from C3; symbol Device:C -> lib:C
- Cboot1: renamed from Cboot; symbol Device:C -> lib:C
- D1: symbol Device:LED -> lib:LED
- IC1: renamed from IC2; symbol DC-DC converters:TPS56637RPAR -> lib:TPS56637RPAR_1
- J1: symbol Connector_Generic:Conn_01x02 -> lib:Conn_01x02
- L1: symbol Device:L -> lib:L
- R4: renamed from R2; symbol Device:R -> lib:R
- R5: renamed from R3; symbol Device:R -> lib:R
- R6: renamed from R4; symbol Device:R -> lib:R
- R7: renamed from R1; symbol Device:R -> lib:R
Connections:
- net +16V: now also R7.2, R2.1, R8.2
- net GND: now also Q1.2 (S), R3.2
- net at D1.1 (K): now also Q1.3 (D); no longer IC1.4 (PG)
- net at D1.2 (A): now also R8.1; no longer R7.1
- net at C4.1, J1.1 (Pin_1), L1.2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: no longer R7.2
- net at IC1.1 (EN): now also R1.2, R2.2, R3.1
- new net gas_en: R1.1
- new net pg_gas: IC1.4 (PG), Q1.1 (G), R7.1
Other:
- moved on the sheet: C1, C2, C3, C4, Cboot1, D1, IC1, J1, L1, R4, R5, R6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

Commit message: Clean up
Other:
- title: (none) -> Robot power supply
Changed lines of the file:
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@@
 	(generator_version "9.0")
 	(paper "A4")
+	(title_block
+		(title "Robot power supply")
+		(date "2026-01-24")
+		(rev "rev 1.0")
+	)
 	(junction
 		(at 81.28 96.52)
