File: MCU.kicad_sch (KiCad schematic)
At the start: 40 parts, among them J1 Conn_01x04, J2 PinHeader_2x5_P1.27mm_SMD, SW3 SW_Push, U3 STM32U585CIT3, U8 SI2301CDS-T1-GE3, U9 527450897, Y1 Oscillator_40MHz_YIC_OSC-S5

Commit message: Charging circuit, new block diagram, MCU and display
Parts:
- removed C21, C22: 1uF, PCM_JLCPCB:C_0402, symbol PCM_JLCPCB-Capacitors:0402,1uF
- removed C23, C25: 100nF, PCM_JLCPCB:C_0402, symbol PCM_JLCPCB-Capacitors:0402,100nF,(2)
- removed LS1: PS1240P02BT, Hardware Components Footprints:Buzzer_THT_PS1240P02BT, symbol Hardware Components:PS1240P02BT
- removed R13, R15, R23, R24: 10kΩ, PCM_JLCPCB:R_0402, symbol PCM_JLCPCB-Resistors:0402,10kΩ
- removed R14: 5.1Ω, PCM_JLCPCB:R_0805, symbol PCM_JLCPCB-Resistors:0805,5.1Ω
- removed R16: 0R, Hardware Components Footprints:R_0402_1005Metric, symbol Device:R_Small
- removed R2: 1k, Resistor_SMD:R_0603_1608Metric_Pad0.98x0.95mm_HandSolder, symbol Device:R_Small
- removed R30, R32: 100Ω, PCM_JLCPCB:R_0402, symbol PCM_JLCPCB-Resistors:0402,100Ω
- removed SW3, SW?: SW_Push, Button_Switch_Keyboard:SW_Cherry_MX_1.00u_PCB, symbol Switch:SW_Push
- removed TP13, TP14: TestPoint, UserLib:TestPoint, symbol Connector:TestPoint
- removed U8: SI2301CDS-T1-GE3, jlc_footprints:SOT-23-3_L3.0-W1.7-P0.95-LS2.9-BR, symbol JLC_imports:SI2301CDS-T1-GE3
- removed U9: 527450897, jlc_footprints:FPC-SMD_527450897, symbol JLC_imports:527450897
- added C45, C46: C_100n_50V_X8L_0402, Hardware Components Footprints:C_0402_1005Metric, symbol lib:C_100n_50V_X8L_0402
- added R64, R66: R_4k7_0402, Hardware Components Footprints:R_0402_1005Metric, symbol lib:R_4k7_0402
- added R67, R68: R_100R_0402, Hardware Components Footprints:R_0402_1005Metric, symbol lib:R_100R_0402
- added R69, R70: R_10k_0.1%_0402, Hardware Components Footprints:R_0402_1005Metric, symbol lib:R_10k_0.1%_0402
- added SW1, SW2: SW_KSC441J70SHLFS_SMD, Hardware Components Footprints:SW_KSC441J70SHLFS_SMD, symbol lib:SW_KSC441J70SHLFS_SMD
- C36: renamed from C1; symbol Hardware Components:C_1u_0402 -> lib:C_1u_0402
- C37: renamed from C4; symbol Hardware Components:C_1u_0402 -> lib:C_1u_0402
- C38: renamed from C6; symbol Hardware Components:C_1u_0402 -> lib:C_1u_0402
- C39: renamed from C7; symbol Hardware Components:C_100n_50V_X8L_0402 -> lib:C_100n_50V_X8L_0402
- C40: renamed from C8; symbol Hardware Components:C_1u_0402 -> lib:C_1u_0402
- C41: renamed from C9; symbol Hardware Components:C_1u_0402 -> lib:C_1u_0402
- C42: renamed from C10; symbol Hardware Components:C_4u7_0402 -> lib:C_4u7_0402
- C43: renamed from C11; symbol Hardware Components:C_1u_0402 -> lib:C_1u_0402
- C44: renamed from C14; symbol Hardware Components:C_1u_0402 -> lib:C_1u_0402
- C47: renamed from C2; symbol Hardware Components:C_1u_0402 -> lib:C_1u_0402
- D6: renamed from D1; symbol Device:LED -> lib:LED
- J7: renamed from J1; symbol Connector_Generic:Conn_01x04 -> lib:Conn_01x04
- J8: renamed from J2; symbol Hardware Components:PinHeader_2x5_P1.27mm_SMD -> lib:PinHeader_2x5_P1.27mm_SMD
- R60: renamed from R1; symbol Hardware Components:R_0R_0201 -> lib:R_0R_0201
- R61: renamed from R2; symbol Device:R_Small -> lib:R_Small
- R62: renamed from R1; symbol Hardware Components:R_10k_0402 -> lib:R_10k_0402
- R63: renamed from R7; symbol Hardware Components:R_4k7_0402 -> lib:R_4k7_0402
- R65: renamed from R8; symbol Hardware Components:R_4k7_0402 -> lib:R_4k7_0402
- U3: symbol MCU_ST_STM32U5:STM32U585CITx -> lib:STM32U585CITx
- Y1: symbol Hardware Components:Oscillator_40MHz_YIC_OSC-S5 -> lib:Oscillator_40MHz_YIC_OSC-S5
Connections:
- net +3V3: now also R64.2, R66.2, R69.2, R70.2
- net BTN1: now also U3.29 (PA8), R68.1; no longer U3.25 (PB12)
- net BTN2: now also U3.30 (PA9), R67.1; no longer U3.26 (PB13)
- net GND: now also C45.1, C46.1, SW1.3, SW1.4, SW2.3, SW2.4
- net CHG_INT#: now reaches U3.10 (PA0)
- net CHG_QON#: now reaches U3.14 (PA4)
- net ~{ST_ALERT}: now reaches U3.15 (PA5)
- net CHG_CE#: now reaches U3.16 (PA6)
- net SCL{I2C_{2}}: now reaches U3.21 (PB10)
- net SCL{I2C_{2}}: now also R66.1
- net SDA{I2C_{2}}: now reaches U3.27 (PB14)
- net SDA{I2C_{2}}: now also R64.1
- net romeo_en: now reaches U3.28 (PB15)
- net BTP_INT: now reaches U3.40 (PB4)
- net ~{PRES}: now reaches U3.41 (PB5)
- net gas_en: now reaches U3.45 (PB8)
- net motor_en : now reaches U3.46 (PB9)
- new net: C46.2, R68.2, R70.1, SW2.1, SW2.2
- new net: C45.2, R67.2, R69.1, SW1.1, SW1.2
- new net fan_en: U3.25 (PB12)
- no-connect marks 23 -> 12
Other:
- note added: "from arm spec"
- note removed: "From arm.com"
- moved on the sheet: C36, C37, C38, C39, C40, C41, C42, C43, C44, C47, D6, J7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

Commit message: Clean up
Other:
- title: (none) -> Robot power supply
Changed lines of the file:
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@@
 	(generator_version "9.0")
 	(paper "A4")
+	(title_block
+		(title "Robot power supply")
+		(date "2026-01-24")
+		(rev "rev 1.0")
+	)
 	(text "from arm spec\n"
 		(exclude_from_sim no)
