File: MCU.kicad_sch (KiCad schematic)
At the start: 35 parts, among them J7 Conn_01x04, J8 PinHeader_2x5_P1.27mm_SMD, SW1 SW_KSC441J70SHLFS_SMD, SW2 SW_KSC441J70SHLFS_SMD, U3 STM32U585CIT3, Y1 Oscillator_40MHz_YIC_OSC-S5

Commit message: Added routing uC
Parts:
- removed A1: Mech_Adafruit_326_H6.0mm, Hardware Components Footprints:Mech_Adafruit_326_H6.0mm, symbol Hardware Components:Mech_Adafruit_326_H6.0mm
Connections:
- net BTN1: now also U3.31 (PA10); no longer U3.29 (PA8)
- net fan_en: now also U3.28 (PB15); no longer U3.25 (PB12)
- net gas_en: now also U3.29 (PA8); no longer U3.45 (PB8)
- net motor_en : now also U3.25 (PB12); no longer U3.46 (PB9)
- net romeo_en: now also U3.26 (PB13); no longer U3.28 (PB15)
