File: RomeoDC-DC.kicad_sch (KiCad schematic)
At the start: 0 parts

Commit message: Clean up
Other:
- title: (none) -> Robot power supply
Changed lines of the file:
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@@
 	(generator_version "9.0")
 	(paper "A4")
+	(title_block
+		(title "Robot power supply")
+		(date "2026-01-24")
+		(rev "rev 1.0")
+	)
 )
