File: bms.kicad_sch (KiCad schematic)
At the start: 71 parts, among them J5 Screw_Terminal_01x02, J6 Molex_Pico-Clasp_1x7_Horizont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, Q10 CSD17579Q5A, Q11 SiA453EDJ, Q12 CSD17579Q5A, Q13 2N7002K, Q5 DMN2056U, Q6 DMN2056U, Q7 DMN2056U, Q8 DMG2301L, Q9 Si1442DH, U1 BQ29410_TSSOP, U2 BQ40Z50RSMT-R2

Commit message: Clean up
Other:
- title: sniffer robot power managment unit -> Robot power supply
Changed lines of the file:
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@@
 	(paper "A3")
 	(title_block
-		(title "sniffer robot power managment unit")
-		(date "2025-11-15")
-		(rev "Rev 1.0.0")
+		(title "Robot power supply")
+		(date "2026-01-24")
+		(rev "rev 1.0")
 	)
 	(rectangle
