File: bms.kicad_sch (KiCad schematic)
At the start: 0 parts

Commit message: Fixed schematic, basic floor plan
Parts:
- added J4, J5: Conn_01x01, TestPoint:TestPoint_THTPad_D4.0mm_Drill2.0mm, symbol Connector_Generic:Conn_01x01
- added J6: Conn_01x03, Connector_PinHeader_2.54mm:PinHeader_1x05_P2.54mm_Horizontal, symbol Connector_Generic:Conn_01x03
Connections:
- new net +16V: J5.1 (Pin_1)
- new net B1: J6.3 (Pin_3)
- new net B2: J6.2 (Pin_2)
- new net B3: J6.1 (Pin_1)
- new net GND: J4.1 (Pin_1)
