File: charger.kicad_sch (KiCad schematic)
At the start: 43 parts, among them J9 USB-C_CUI_UJC-HP-3-SMT-TR, Q14 SQS401EN-T1_BE3, U6 STUSB4500_QFN, U7 BQ25798RQMR

Commit message: Clean up
Other:
- title: (none) -> Robot power supply
Changed lines of the file:
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@@
 	(generator_version "9.0")
 	(paper "A3")
+	(title_block
+		(title "Robot power supply")
+		(date "2026-01-24")
+		(rev "rev 1.0")
+	)
 	(text "address 0101000(R/W)"
 		(exclude_from_sim no)
