File: robot-pmu-hw.kicad_sch (KiCad schematic)
At the start: 0 parts

Commit message: Charging circuit, new block diagram, MCU and display
Other:
- added sheet BMS (bms.kicad_sch)
- added sheet Charger (charger.kicad_sch)
- added sheet Display (display.kicad_sch)
- added sheet uC (MCU.kicad_sch)
- sheet FanDC-DC ports: added fan_en ; removed none
- sheet GasDC-DC ports: added gas_en; removed none
- sheet MotorDC-DC ports: added motor_en ; removed none
- note added: "I2C ADDRESS TABLE (7-Bit) ------------------------ BQ25798 (Charger) : 0x6B STUSB4500 (USB-PD) : 0x28 (Bin: 0101000) BQ40Z50-R2 (BMS) : 0x0B (8-bit Wr: 0x16)"
- note removed: "DC-DC Enable"
- note removed: "Possibly reduce max amperage and save space ?"
- note removed: "USB PD 20V?"

Commit message: Clean up
Other:
- title: (none) -> Robot power supply
