File: display.kicad_sch (KiCad schematic)
At the start: 10 parts, among them U4 SI2301CDS-T1-GE3, U5 527450897

Commit message: Clean up
Other:
- title: (none) -> Robot power supply
Changed lines of the file:
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@@
 	(generator_version "9.0")
 	(paper "A4")
+	(title_block
+		(title "Robot power supply")
+		(date "2026-01-24")
+		(rev "rev 1.0")
+	)
 	(junction
 		(at 144.78 83.82)

Commit message: Fixed schematic, basic floor plan
Parts:
- removed C48, C49: C_1u_0402, Hardware Components Footprints:C_0402_1005Metric, symbol lib:C_1u_0402
- removed R71, R72: R_10k_0.1%_0402, Hardware Components Footprints:R_0402_1005Metric, symbol lib:R_10k_0.1%_0402
- removed R73: R_5R1_0603, Hardware Components Footprints:R_0603_1608Metric, symbol lib:R_5R1_0603
- removed R74: 0R, Hardware Components Footprints:R_0402_1005Metric, symbol lib:R_Small
- removed TP8, TP9: TestPoint, UserLib:TestPoint, symbol lib:TestPoint
- removed U4: SI2301CDS-T1-GE3, jlc_footprints:SOT-23-3_L3.0-W1.7-P0.95-LS2.9-BR, symbol lib:SI2301CDS-T1-GE3
- removed U5: 527450897, jlc_footprints:FPC-SMD_527450897, symbol lib:527450897
